Commit message: fixed urdf bug

File: src/robotic_arm/urdf/robotic_arm.urdf (robot description, URDF)
Before this commit: robot robotic_arm, 8 links, 7 joints
Joints:
- joint shift_joint: limit lower=0 upper=0 effort=0 velocity=0 -> lower=-0.2 upper=0.2 effort=0 velocity=0

File: src/robotic_arm_moveit_config/config/robotic_arm.ros2_control.xacro (robot description, xacro)
@@ -2,5 +2,5 @@
 <robot xmlns:xacro="http://www.ros.org/wiki/xacro">
     <xacro:macro name="robotic_arm_ros2_control" params="name initial_positions_file">
-        <xacro:property name="initial_positions" value="${load_yaml(initial_positions_file)['initial_positions']}"/>
+        <xacro:property name="initial_positions" value="${xacro.load_yaml(initial_positions_file)['initial_positions']}"/>
         <ros2_control name="${name}" type="system">
             <hardware>
